File: led_mapper_eorspec/rhombus/single_net_reverse_cols.kicad_sch (KiCad schematic)
At the start: 529 parts

Commit message: Complete single-net schematic, led placement and vertical tracks
Parts:
- gave numbers to parts that had none: 528
- renumbered D1610 to D552
