File: led_mapper_eorspec/_misc/rhombus/led_mapper_eorspec.kicad_pcb (KiCad board)
At the start: 4 copper layers, 116 x 67 mm, 1025 parts, among them J1 Conn_02x12_Top_Bottom

Commit message: Move misc. files to _misc directory
Routing:
- net /P7: track 210.4 -> 229.4 mm
- net /P6: track 210.7 -> 229.6 mm
- net /P4: track 211.3 -> 230.2 mm
- net /P5: track 211.0 -> 229.8 mm
- net /P8: track 214.3 -> 233.1 mm
- net /P2: track 210.0 -> 228.8 mm
- net /P3: track 211.6 -> 230.4 mm
- net /P1: track 214.3 -> 233.1 mm
- net /P9: track 225.4 -> 226.5 mm
Changed lines of the file:
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@@
 	)
 	(segment
+		(start 60.068306 59.566862)
+		(end 59.047499 59.574951)
+		(width 0.2)
+		(layer "In1.Cu")
+		(net "/P2")
+	)
+	(segment
+		(start 69.497499 45.095007)
+		(end 68.464113 45.102448)
+		(width 0.2)
+		(layer "In1.Cu")
+		(net "/P2")
+	)
+	(segment
+		(start 68.464113 45.102448)
+		(end 60.068306 59.566862)
+		(width 0.2)
+		(layer "In1.Cu")
+		(net "/P2")
+	)
+	(segment
 		(start 88.425 22.470091)
 		(end 88.83 20.660098)
@@
 	)
 	(segment
+		(start 80.930643 37.884065)
+		(end 72.640753 52.391373)
+		(width 0.2)
+		(layer "In1.Cu")
+		(net "/P6")
+	)
+	(segment
+		(start 72.640753 52.391373)
+		(end 71.587499 52.334979)
+		(width 0.2)
+		(layer "In1.Cu")
+		(net "/P6")
+	)
+	(segment
+		(start 82.037499 37.855035)
+		(end 80.930643 37.884065)
+		(width 0.2)
+		(layer "In1.Cu")
+		(net "/P6")
+	)
+	(segment
 		(start 76.93 46)
 		(end 76.812499 46.905)
@@
 	)
 	(segment
+		(start 56.867676 61.380278)
+		(end 55.912499 61.384944)
+		(width 0.2)
+		(layer "In1.Cu")
+		(net "/P1")
+	)
+	(segment
+		(start 66.362499 46.905)
+		(end 65.313066 46.903382)
+		(width 0.2)
+		(layer "In1.Cu")
+		(net "/P1")
+	)
+	(segment
+		(start 65.313066 46.903382)
+		(end 56.867676 61.380278)
+		(width 0.2)
+		(layer "In1.Cu")
+		(net "/P1")
+	)
+	(segment
 		(start 9.005 69.529909)
 		(end 8.887499 70.434909)
@@
 	)
 	(segment
+		(start 88.307499 34.235049)
+		(end 87.282637 34.25051)
+		(width 0.2)
+		(layer "In1.Cu")
+		(net "/P8")
+	)
+	(segment
+		(start 78.885086 48.730902)
+		(end 77.857499 48.714993)
+		(width 0.2)
+		(layer "In1.Cu")
+		(net "/P8")
+	)
+	(segment
+		(start 87.282637 34.25051)
+		(end 78.885086 48.730902)
+		(width 0.2)
+		(layer "In1.Cu")
+		(net "/P8")
+	)
+	(segment
 		(start 66.48 56.859958)
 		(end 66.362499 57.764958)
@@
 	)
 	(segment
+		(start 63.260502 57.770549)
+		(end 62.182499 57.764958)
+		(width 0.2)
+		(layer "In1.Cu")
+		(net "/P3")
+	)
+	(segment
+		(start 71.658053 43.3081)
+		(end 63.260502 57.770549)
+		(width 0.2)
+		(layer "In1.Cu")
+		(net "/P3")
+	)
+	(segment
+		(start 72.632499 43.285014)
+		(end 71.658053 43.3081)
+		(width 0.2)
+		(layer "In1.Cu")
+		(net "/P3")
+	)
+	(segment
 		(start 39.715 47.809993)
 		(end 29.265 65.909923)
@@
 	)
 	(segment
+		(start 30.832499 46.905)
+		(end 31.355 47.809993)
+		(width 0.2)
+		(layer "F.Cu")
+		(net "/P9")
+	)
+	(segment
 		(start 24.68 46)
 		(end 24.562499 46.905)
@@
 	)
 	(segment
+		(start 85.172499 36.045042)
+		(end 84.10664 36.026915)
+		(width 0.2)
+		(layer "In1.Cu")
+		(net "/P7")
+	)
+	(segment
+		(start 75.789835 50.641883)
+		(end 74.722499 50.524986)
+		(width 0.2)
+		(layer "In1.Cu")
+		(net "/P7")
+	)
+	(segment
+		(start 84.10664 36.026915)
+		(end 75.789835 50.641883)
+		(width 0.2)
+		(layer "In1.Cu")
+		(net "/P7")
+	)
+	(segment
 		(start 20.5 49.619986)
 		(end 20.382499 50.524986)
@@
 	)
 	(segment
+		(start 78.902499 39.665028)
+		(end 77.866499 39.674222)
+		(width 0.2)
+		(layer "In1.Cu")
+		(net "/P5")
+	)
+	(segment
+		(start 77.866499 39.674222)
+		(end 69.463231 54.166238)
+		(width 0.2)
+		(layer "In1.Cu")
+		(net "/P5")
+	)
+	(segment
+		(start 69.463231 54.166238)
+		(end 68.452499 54.144972)
+		(width 0.2)
+		(layer "In1.Cu")
+		(net "/P5")
+	)
+	(segment
 		(start 58.12 42.380014)
 		(end 58.002499 43.285014)
@@
 		(net "/P4")
 	)
+	(segment
+		(start 66.382668 55.9762)
+		(end 65.317499 55.954965)
+		(width 0.2)
+		(layer "In1.Cu")
+		(net "/P4")
+	)
+	(segment
+		(start 75.767499 41.475021)
+		(end 74.735925 41.475949)
+		(width 0.2)
+		(layer "In1.Cu")
+		(net "/P4")
+	)
+	(segment
+		(start 74.735925 41.475949)
+		(end 66.382668 55.9762)
+		(width 0.2)
+		(layer "In1.Cu")
+		(net "/P4")
+	)
